File: kicad/tenshi.kicad_pcb (KiCad board)
At the start: 2 copper layers, 262.6 x 94.5 mm, 76 parts

Commit message: Add logo
Parts:
- added G***: LOGO, Aafootprints:wing-right, F.Cu at (227.3, 81.1)
- added G***: LOGO, Aafootprints:wing-left, F.Cu at (67.9, 81.1)
- REF** (x2): footprint footprints:HRO-TYPE-C-31-M-12 -> Aafootprints:HRO-TYPE-C-31-M-12

Commit message: Add logo
Parts:
- added G***: LOGO, Aafootprints:logo, F.Cu at (242.8, 84.8)
- added G***: LOGO, Aafootprints:logo, F.Cu at (52.4, 84.8)

Commit message: Add url
Parts:
- added G***: LOGO, Aafootprints:wing-right-large, F.Cu at (226.3, 56.9)
- added G***: LOGO, Aafootprints:url, F.Cu at (84.1, 85.6)
- added G***: LOGO, Aafootprints:wing-left-large, F.Cu at (69.0, 56.9)
- added G***: LOGO, Aafootprints:url, F.Cu at (211.0, 85.6)
